File: hardware/axis.kicad_pcb (KiCad board)
At the start: 4 copper layers, 66 x 17.5 mm, 43 parts, among them J101 Cortex, J102 DX07S016JA3, SW101 SKSG, SW102 SKSG, U101 BHI160, U102 ATSAMD51G, U103 BMM150, U104 TPS78433QWDRBRQ1, Y101 32k768

Commit message: Refresh
Parts:
- C101, C102, C103, C104, C105, C106, C107, C108, C109, C110: footprint V2_Capacitor_SMD:C_0603 -> V2_Capacitor_SMD:C_1608
- C111, C112: footprint V2_Capacitor_SMD:C_0805 -> V2_Capacitor_SMD:C_2012
- D101: footprint V2_LED:LED_0603 -> V2_LED:LED_1608
- R101, R102, R103, R104, R105, R106, R107, R108: footprint V2_Resistor_SMD:R_0603 -> V2_Resistor_SMD:R_1608
Changed lines of the file:
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@@
 	(paper "A4")
 	(title_block
-		(date "2026-04-14")
+		(date "2026-05-19")
 		(rev "2026-01-14")
 	)
@@
 		)
 	)
-	(footprint "V2_Resistor_SMD:R_0603"
+	(footprint "V2_Resistor_SMD:R_1608"
 		(layer "F.Cu")
 		(at 125 112.75 180)
@@
 			)
 		)
-		(property "Id" "Resistor:0603_5k1"
+		(property "Id" "Resistor:1608_5k1"
 			(at 0 0 180)
 			(unlocked yes)
@@
 		)
 	)
-	(footprint "V2_Capacitor_SMD:C_0603"
+	(footprint "V2_Capacitor_SMD:C_1608"
 		(layer "F.Cu")
 		(at 175.25 109.75)
@@
 			)
 		)
-		(property "Id" "Capacitor:0603_0u47"
+		(property "Id" "Capacitor:1608_0u47"
 			(at 0 0 0)
 			(unlocked yes)
@@
 		(embedded_fonts no)
 	)
-	(footprint "V2_Resistor_SMD:R_0603"
+	(footprint "V2_Resistor_SMD:R_1608"
 		(layer "F.Cu")
 		(at 175.25 102.75)
@@
 			)
 		)
-		(property "Id" "Resistor:0603_2k7"
+		(property "Id" "Resistor:1608_2k7"
 			(at 0 0 0)
 			(unlocked yes)
@@
 		)
 	)
-	(footprint "V2_Capacitor_SMD:C_0603"
+	(footprint "V2_Capacitor_SMD:C_1608"
 		(layer "F.Cu")
 		(at 135.25 104.25 180)
@@
 			)
 		)
-		(property "Id" "Capacitor:0603_18p"
+		(property "Id" "Capacitor:1608_18p"
 			(at 0 0 180)
 			(unlocked yes)
@@
 		)
 	)
-	(footprint "V2_Capacitor_SMD:C_0603"
+	(footprint "V2_Capacitor_SMD:C_1608"
 		(layer "F.Cu")
 		(at 172 109.75 180)
@@
 			)
 		)
-		(property "Id" "Capacitor:0603_1u"
+		(property "Id" "Capacitor:1608_1u"
 			(at 0 0 180)
 			(unlocked yes)
@@
 		)
 	)
-	(footprint "V2_Capacitor_SMD:C_0603"
+	(footprint "V2_Capacitor_SMD:C_1608"
 		(layer "F.Cu")
 		(at 175.25 111.75 180)
@@
 			)
 		)
-		(property "Id" "Capacitor:0603_10u"
+		(property "Id" "Capacitor:1608_10u"
 			(at 0 0 180)
 			(unlocked yes)
@@
 		)
 	)
-	(footprint "V2_Capacitor_SMD:C_0603"
+	(footprint "V2_Capacitor_SMD:C_1608"
 		(layer "F.Cu")
 		(at 138.5 106.75 90)
@@
 			)
 		)
-		(property "Id" "Capacitor:0603_1u"
+		(property "Id" "Capacitor:1608_1u"
 			(at 0 0 90)
 			(unlocked yes)
@@
 		(embedded_fonts no)
 	)
-	(footprint "V2_Resistor_SMD:R_0603"
+	(footprint "V2_Resistor_SMD:R_1608"
 		(layer "F.Cu")
 		(at 125 99.75 180)
@@
 			)
 		)
-		(property "Id" "Resistor:0603_5k1"
+		(property "Id" "Resistor:1608_5k1"
 			(at 0 0 180)
 			(unlocked yes)
@@
 		(embedded_fonts no)
 	)
-	(footprint "V2_Capacitor_SMD:C_0603"
+	(footprint "V2_Capacitor_SMD:C_1608"
 		(layer "F.Cu")
 		(at 150.25 102.75)
@@
 			)
 		)
-		(property "Id" "Capacitor:0603_1u"
+		(property "Id" "Capacitor:1608_1u"
 			(at 0 0 0)
 			(unlocked yes)
@@
 		(embedded_fonts no)
 	)
-	(footprint "V2_Capacitor_SMD:C_0603"
+	(footprint "V2_Capacitor_SMD:C_1608"
 		(layer "F.Cu")
 		(at 144 111.5)
@@
 			)
 		)
-		(property "Id" "Capacitor:0603_1u"
+		(property "Id" "Capacitor:1608_1u"
 			(at 0 0 0)
 			(unlocked yes)
@@
 		)
 	)
-	(footprint "V2_Capacitor_SMD:C_0603"
+	(footprint "V2_Capacitor_SMD:C_1608"
 		(layer "F.Cu")
 		(at 135.25 102.25 180)
@@
 			)
 		)
-		(property "Id" "Capacitor:0603_18p"
+		(property "Id" "Capacitor:1608_18p"
 			(at 0 0 180)
 			(unlocked yes)
@@
 		)
 	)
-	(footprint "V2_Capacitor_SMD:C_0805"
+	(footprint "V2_Capacitor_SMD:C_2012"
 		(layer "F.Cu")
 		(at 138.5 111.25 90)
@@
 			)
 		)
-		(property "Id" "Capacitor:0805_10u"
+		(property "Id" "Capacitor:2012_10u"
 			(at 0 0 90)
 			(unlocked yes)
@@
 		)
 	)
-	(footprint "V2_Resistor_SMD:R_0603"
+	(footprint "V2_Resistor_SMD:R_1608"
 		(layer "F.Cu")
 		(at 150.25 100.75)
@@
 			)
 		)
-		(property "Id" "Resistor:0603_100k"
+		(property "Id" "Resistor:1608_100k"
 			(at 0 0 0)
 			(unlocked yes)
@@
 		)
 	)
-	(footprint "V2_Capacitor_SMD:C_0603"
+	(footprint "V2_Capacitor_SMD:C_1608"
 		(layer "F.Cu")
 		(at 145.5 100.75 180)
@@
 			)
 		)
-		(property "Id" "Capacitor:0603_10u"
+		(property "Id" "Capacitor:1608_10u"
 			(at 0 0 180)
 			(unlocked yes)
@@
 		)
 	)
-	(footprint "V2_Resistor_SMD:R_0603"
+	(footprint "V2_Resistor_SMD:R_1608"
 		(layer "F.Cu")
 		(at 163.5 101.25)
@@
 			)
 		)
-		(property "Id" "Resistor:0603_2k7"
+		(property "Id" "Resistor:1608_2k7"
 			(at 0 0 0)
 			(unlocked yes)
@@
 		)
 	)
-	(footprint "V2_Resistor_SMD:R_0603"
+	(footprint "V2_Resistor_SMD:R_1608"
 		(layer "F.Cu")
 		(at 158.75 100.5 180)
@@
 			)
 		)
-		(property "Id" "Resistor:0603_330R"
+		(property "Id" "Resistor:1608_330R"
 			(at 0 0 180)
 			(unlocked yes)
@@
 		)
 	)
-	(footprint "V2_Resistor_SMD:R_0603"
+	(footprint "V2_Resistor_SMD:R_1608"
 		(layer "F.Cu")
 		(at 178.75 102.75 180)
@@
 			)
 		)
-		(property "Id" "Resistor:0603_2k7"
+		(property "Id" "Resistor:1608_2k7"
 			(at 0 0 180)
 			(unlocked yes)
@@
 		)
 	)
-	(footprint "V2_Capacitor_SMD:C_0603"
+	(footprint "V2_Capacitor_SMD:C_1608"
 		(layer "F.Cu")
 		(at 142 100.75 180)
@@
 			)
 		)
-		(property "Id" "Capacitor:0603_1u"
+		(property "Id" "Capacitor:1608_1u"
 			(at 0 0 180)
 			(unlocked yes)
@@
 		)
 	)
-	(footprint "V2_LED:LED_0603"
+	(footprint "V2_LED:LED_1608"
 		(layer "F.Cu")
 		(at 158.75 102 180)
@@
 			)
 		)
-		(property "Id" "LED:0603_Orange"
+		(property "Id" "LED:1608_Orange"
 			(at 0 0 180)
 			(unlocked yes)
@@
 		)
 	)
-	(footprint "V2_Resistor_SMD:R_0603"
+	(footprint "V2_Resistor_SMD:R_1608"
 		(layer "F.Cu")
 		(at 163.5 103.25)
@@
 			)
 		)
-		(property "Id" "Resistor:0603_2k7"
+		(property "Id" "Resistor:1608_2k7"
 			(at 0 0 0)
 			(unlocked yes)
@@
 		(embedded_fonts no)
 	)
-	(footprint "V2_Capacitor_SMD:C_0805"
+	(footprint "V2_Capacitor_SMD:C_2012"
 		(layer "F.Cu")
 		(at 132 111.25 90)
@@
 			)
 		)
-		(property "Id" "Capacitor:0805_10u"
+		(property "Id" "Capacitor:2012_10u"
 			(at 0 0 90)
 			(unlocked yes)
@@
 		(layer "F.Cu")
 		(hatch none 0.1)
-		(priority 30032)
+		(priority 30029)
 		(attr
 			(teardrop
@@
 		(polygon
 			(pts
-				(xy 139.745677 105.625) (xy 139.766353 105.620399) (xy 139.76689 105.608189) (xy 139.728493 105.573671)
-				(xy 139.610415 105.51724) (xy 139.562623 105.50843) (xy 139.532979 105.518689) (xy 139.529323 105.543895)
-				(xy 139.974 105.5) (xy 139.529323 105.543895) (xy 139.538372 105.565093) (xy 139.55399 105.576049)
-				(xy 139.599191 105.572546) (xy 139.677112 105.52781) (xy 139.763213 105.43898) (xy 139.778382 105.405801)
-				(xy 139.773106 105.38279) (xy 139.745677 105.375)
+				(xy 139.499058 105.625) (xy 139.542474 105.629861) (xy 139.569912 105.64389) (xy 139.585575 105.656688)
+				(xy 139.624997 105.687081) (xy 139.755323 105.5) (xy 139.624997 105.312919) (xy 139.585575 105.343312)
+				(xy 139.551875 105.366768) (xy 139.499058 105.375)
 			)
 		)
@@
 		(layer "F.Cu")
 		(hatch none 0.1)
-		(priority 30003)
+		(priority 30032)
 		(attr
 			(teardrop
@@
 		(polygon
 			(pts
-				(xy 140.195677 105.375) (xy 140.105298 105.370368) (xy 140.040248 105.357943) (xy 139.967303 105.331993)
-				(xy 139.896246 105.305588) (xy 139.793895 105.279323) (xy 139.744677 105.5) (xy 139.793895 105.720677)
-				(xy 139.94627 105.676376) (xy 139.967302 105.668006) (xy 140.05837 105.637534) (xy 140.195677 105.625)
+				(xy 139.745677 105.625) (xy 139.766353 105.620399) (xy 139.76689 105.608189) (xy 139.728493 105.573671)
+				(xy 139.610415 105.51724) (xy 139.562623 105.50843) (xy 139.532979 105.518689) (xy 139.529323 105.543895)
+				(xy 139.974 105.5) (xy 139.529323 105.543895) (xy 139.538372 105.565093) (xy 139.55399 105.576049)
+				(xy 139.599191 105.572546) (xy 139.677112 105.52781) (xy 139.763213 105.43898) (xy 139.778382 105.405801)
+				(xy 139.773106 105.38279) (xy 139.745677 105.375)
 			)
 		)
@@
 		(layer "F.Cu")
 		(hatch none 0.1)
-		(priority 30029)
+		(priority 30003)
 		(attr
 			(teardrop
@@
 		(polygon
 			(pts
-				(xy 139.499058 105.625) (xy 139.542474 105.629861) (xy 139.569912 105.64389) (xy 139.585575 105.656688)
-				(xy 139.624997 105.687081) (xy 139.755323 105.5) (xy 139.624997 105.312919) (xy 139.585575 105.343312)
-				(xy 139.551875 105.366768) (xy 139.499058 105.375)
+				(xy 140.195677 105.375) (xy 140.105298 105.370368) (xy 140.040248 105.357943) (xy 139.967303 105.331993)
+				(xy 139.896246 105.305588) (xy 139.793895 105.279323) (xy 139.744677 105.5) (xy 139.793895 105.720677)
+				(xy 139.94627 105.676376) (xy 139.967302 105.668006) (xy 140.05837 105.637534) (xy 140.195677 105.625)
 			)
 		)
@@
 		(layer "F.Cu")
 		(hatch none 0.1)
-		(priority 30001)
+		(priority 30000)
 		(attr
 			(teardrop
@@
 		(polygon
 			(pts
-				(xy 144.4 102.445677) (xy 144.404725 102.331788) (xy 144.417796 102.253944) (xy 144.432926 102.197771)
-				(xy 144.470677 102.043895) (xy 144.25 101.994677) (xy 144.029323 102.043895) (xy 144.067075 102.197773)
-				(xy 144.091021 102.298464) (xy 144.1 102.445677)
+				(xy 144.1 101.554323) (xy 144.095275 101.66821) (xy 144.082204 101.746053) (xy 144.067075 101.802226)
+				(xy 144.029323 101.956105) (xy 144.25 102.005323) (xy 144.470677 101.956105) (xy 144.432925 101.802228)
+				(xy 144.408979 101.701536) (xy 144.4 101.554323)
 			)
 		)
@@
 		(layer "F.Cu")
 		(hatch none 0.1)
-		(priority 30000)
+		(priority 30001)
 		(attr
 			(teardrop
@@
 		(polygon
 			(pts
-				(xy 144.1 101.554323) (xy 144.095275 101.66821) (xy 144.082204 101.746053) (xy 144.067075 101.802226)
-				(xy 144.029323 101.956105) (xy 144.25 102.005323) (xy 144.470677 101.956105) (xy 144.432925 101.802228)
-				(xy 144.408979 101.701536) (xy 144.4 101.554323)
+				(xy 144.4 102.445677) (xy 144.404725 102.331788) (xy 144.417796 102.253944) (xy 144.432926 102.197771)
+				(xy 144.470677 102.043895) (xy 144.25 101.994677) (xy 144.029323 102.043895) (xy 144.067075 102.197773)
+				(xy 144.091021 102.298464) (xy 144.1 102.445677)
 			)
 		)

Commit message: Refresh
Parts:
- INFO102: value Layer_Numbers -> Layer_Numbers-4; footprint V2_Production:Layer_Numbers -> V2_Production:Layer_Numbers-4
Routing:
- net /USB+: track 36.1 -> 35.6 mm
- net /USB-: track 36.5 -> 37.0 mm
