File: hardware/axis.kicad_pcb (KiCad board)
At the start: 4 copper layers, 66 x 17.5 mm, 43 parts, among them J101 Cortex, J102 DX07S016JA3, SW101 SKSG, SW102 SKSG, U101 BHI160, U102 ATSAMD51G, U103 BMM150, U104 TPS78433QWDRBRQ1, Y101 32k768

Commit message: Rounded edge
Parts:
- moved ICON101 14.5 mm to (182.8, 106.2)
- moved ICON102 10.2 mm to (180.5, 110.5)
- moved FID103 5.00 mm to (177.0, 114.0)
Routing:
- net +3V3: track 117.2 -> 115.2 mm
- net /Interrupt: track 45.2 -> 43.8 mm
- net /USB+: track 35.6 -> 34.3 mm
- net /USB-: track 37.0 -> 35.9 mm
- net /Button: track 23.5 -> 23.0 mm
- net GND: track 30.4 -> 29.9 mm, vias 67 -> 72
Other:
- board size 66 x 17.5 mm -> 70 x 17.5 mm
