File: hardware/axis.kicad_sch (KiCad schematic)
At the start: 43 parts, among them J101 Cortex, J102 DX07S016JA3, SW101 SKSG, SW102 SKSG, U101 BHI160, U102 ATSAMD51G, U103 BMM150, U104 TPS78433QWDRBRQ1, Y101 32k768

Commit message: Good Bye Imperial
Parts:
- C101, C102: footprint V2_Capacitor_SMD:C_0603 -> V2_Capacitor_SMD:C_1608; symbol V2_Capacitor:0603_18p -> V2_Capacitor:1608_18p
- C103, C104: footprint V2_Capacitor_SMD:C_0603 -> V2_Capacitor_SMD:C_1608; symbol V2_Capacitor:0603_10u -> V2_Capacitor:1608_10u
- C105: footprint V2_Capacitor_SMD:C_0603 -> V2_Capacitor_SMD:C_1608; symbol V2_Capacitor:0603_0u47 -> V2_Capacitor:1608_0u47
- C106, C107, C108, C109, C110: footprint V2_Capacitor_SMD:C_0603 -> V2_Capacitor_SMD:C_1608; symbol V2_Capacitor:0603_1u -> V2_Capacitor:1608_1u
- C111, C112: footprint V2_Capacitor_SMD:C_0805 -> V2_Capacitor_SMD:C_2012; symbol V2_Capacitor:0805_10u -> V2_Capacitor:2012_10u
- D101: symbol V2_LED:0603_Orange -> V2_LED:1608_Orange
- R101, R102, R104, R105: footprint V2_Resistor_SMD:R_0603 -> V2_Resistor_SMD:R_1608; symbol V2_Resistor:0603_2k7 -> V2_Resistor:1608_2k7
- R103: footprint V2_Resistor_SMD:R_0603 -> V2_Resistor_SMD:R_1608; symbol V2_Resistor:0603_100k -> V2_Resistor:1608_100k
- R106: footprint V2_Resistor_SMD:R_0603 -> V2_Resistor_SMD:R_1608; symbol V2_Resistor:0603_330R -> V2_Resistor:1608_330R
- R107, R108: footprint V2_Resistor_SMD:R_0603 -> V2_Resistor_SMD:R_1608; symbol V2_Resistor:0603_5k1 -> V2_Resistor:1608_5k1
Changed lines of the file:
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@@
 	)
 	(symbol
-		(lib_id "V2_Resistor:0603_5k1")
+		(lib_id "V2_Resistor:1608_5k1")
 		(at 213.36 95.25 90)
 		(unit 1)
@@
 			)
 		)
-		(property "Footprint" "V2_Resistor_SMD:R_0603"
+		(property "Footprint" "V2_Resistor_SMD:R_1608"
 			(at 229.108 95.25 0)
 			(hide yes)
@@
 	)
 	(symbol
-		(lib_id "V2_Capacitor:0603_1u")
+		(lib_id "V2_Capacitor:1608_1u")
 		(at 115.57 24.13 0)
 		(unit 1)
@@
 			)
 		)
-		(property "Footprint" "V2_Capacitor_SMD:C_0603"
+		(property "Footprint" "V2_Capacitor_SMD:C_1608"
 			(at 115.57 41.148 0)
 			(hide yes)
@@
 	)
 	(symbol
-		(lib_id "V2_Capacitor:0603_1u")
+		(lib_id "V2_Capacitor:1608_1u")
 		(at 148.59 165.1 0)
 		(unit 1)
@@
 			)
 		)
-		(property "Footprint" "V2_Capacitor_SMD:C_0603"
+		(property "Footprint" "V2_Capacitor_SMD:C_1608"
 			(at 148.59 182.118 0)
 			(hide yes)
@@
 	)
 	(symbol
-		(lib_id "V2_Resistor:0603_2k7")
+		(lib_id "V2_Resistor:1608_2k7")
 		(at 33.02 157.48 0)
 		(unit 1)
@@
 			)
 		)
-		(property "Footprint" "V2_Resistor_SMD:R_0603"
+		(property "Footprint" "V2_Resistor_SMD:R_1608"
 			(at 33.02 173.228 0)
 			(hide yes)
@@
 	)
 	(symbol
-		(lib_id "V2_LED:0603_Orange")
+		(lib_id "V2_LED:1608_Orange")
 		(at 127 54.61 180)
 		(unit 1)
@@
 	)
 	(symbol
-		(lib_id "V2_Capacitor:0805_10u")
+		(lib_id "V2_Capacitor:2012_10u")
 		(at 205.74 43.18 0)
 		(unit 1)
@@
 			)
 		)
-		(property "Footprint" "V2_Capacitor_SMD:C_0805"
+		(property "Footprint" "V2_Capacitor_SMD:C_2012"
 			(at 205.74 60.198 0)
 			(hide yes)
@@
 	)
 	(symbol
-		(lib_id "V2_Resistor:0603_2k7")
+		(lib_id "V2_Resistor:1608_2k7")
 		(at 83.82 167.64 0)
 		(unit 1)
@@
 			)
 		)
-		(property "Footprint" "V2_Resistor_SMD:R_0603"
+		(property "Footprint" "V2_Resistor_SMD:R_1608"
 			(at 83.82 183.388 0)
 			(hide yes)
@@
 	)
 	(symbol
-		(lib_id "V2_Resistor:0603_2k7")
+		(lib_id "V2_Resistor:1608_2k7")
 		(at 30.48 157.48 0)
 		(unit 1)
@@
 			)
 		)
-		(property "Footprint" "V2_Resistor_SMD:R_0603"
+		(property "Footprint" "V2_Resistor_SMD:R_1608"
 			(at 30.48 173.228 0)
 			(hide yes)
@@
 	)
 	(symbol
-		(lib_id "V2_Capacitor:0805_10u")
+		(lib_id "V2_Capacitor:2012_10u")
 		(at 180.34 43.18 0)
 		(unit 1)
@@
 			)
 		)
-		(property "Footprint" "V2_Capacitor_SMD:C_0805"
+		(property "Footprint" "V2_Capacitor_SMD:C_2012"
 			(at 180.34 60.198 0)
 			(hide yes)
@@
 	)
 	(symbol
-		(lib_id "V2_Capacitor:0603_18p")
+		(lib_id "V2_Capacitor:1608_18p")
 		(at 36.83 46.99 0)
 		(unit 1)
@@
 			)
 		)
-		(property "Footprint" "V2_Capacitor_SMD:C_0603"
+		(property "Footprint" "V2_Capacitor_SMD:C_1608"
 			(at 36.83 64.008 0)
 			(hide yes)
@@
 	)
 	(symbol
-		(lib_id "V2_Capacitor:0603_10u")
+		(lib_id "V2_Capacitor:1608_10u")
 		(at 63.5 24.13 0)
 		(unit 1)
@@
 			)
 		)
-		(property "Footprint" "V2_Capacitor_SMD:C_0603"
+		(property "Footprint" "V2_Capacitor_SMD:C_1608"
 			(at 63.5 41.148 0)
 			(hide yes)
@@
 	)
 	(symbol
-		(lib_id "V2_Capacitor:0603_18p")
+		(lib_id "V2_Capacitor:1608_18p")
 		(at 31.75 46.99 0)
 		(unit 1)
@@
 			)
 		)
-		(property "Footprint" "V2_Capacitor_SMD:C_0603"
+		(property "Footprint" "V2_Capacitor_SMD:C_1608"
 			(at 31.75 64.008 0)
 			(hide yes)
@@
 	)
 	(symbol
-		(lib_id "V2_Capacitor:0603_0u47")
+		(lib_id "V2_Capacitor:1608_0u47")
 		(at 64.77 168.91 90)
 		(unit 1)
@@
 			)
 		)
-		(property "Footprint" "V2_Capacitor_SMD:C_0603"
+		(property "Footprint" "V2_Capacitor_SMD:C_1608"
 			(at 81.788 168.91 0)
 			(hide yes)
@@
 	)
 	(symbol
-		(lib_id "V2_Resistor:0603_330R")
+		(lib_id "V2_Resistor:1608_330R")
 		(at 134.62 54.61 90)
 		(unit 1)
@@
 			)
 		)
-		(property "Footprint" "V2_Resistor_SMD:R_0603"
+		(property "Footprint" "V2_Resistor_SMD:R_1608"
 			(at 150.368 54.61 0)
 			(hide yes)
@@
 	)
 	(symbol
-		(lib_id "V2_Capacitor:0603_1u")
+		(lib_id "V2_Capacitor:1608_1u")
 		(at 105.41 24.13 0)
 		(unit 1)
@@
 			)
 		)
-		(property "Footprint" "V2_Capacitor_SMD:C_0603"
+		(property "Footprint" "V2_Capacitor_SMD:C_1608"
 			(at 105.41 41.148 0)
 			(hide yes)
@@
 	)
 	(symbol
-		(lib_id "V2_Capacitor:0603_1u")
+		(lib_id "V2_Capacitor:1608_1u")
 		(at 85.09 24.13 0)
 		(unit 1)
@@
 			)
 		)
-		(property "Footprint" "V2_Capacitor_SMD:C_0603"
+		(property "Footprint" "V2_Capacitor_SMD:C_1608"
 			(at 85.09 41.148 0)
 			(hide yes)
@@
 	)
 	(symbol
-		(lib_id "V2_Resistor:0603_5k1")
+		(lib_id "V2_Resistor:1608_5k1")
 		(at 213.36 97.79 90)
 		(unit 1)
@@
 			)
 		)
-		(property "Footprint" "V2_Resistor_SMD:R_0603"
+		(property "Footprint" "V2_Resistor_SMD:R_1608"
 			(at 229.108 97.79 0)
 			(hide yes)
@@
 	)
 	(symbol
-		(lib_id "V2_Resistor:0603_2k7")
+		(lib_id "V2_Resistor:1608_2k7")
 		(at 86.36 167.64 0)
 		(unit 1)
@@
 			)
 		)
-		(property "Footprint" "V2_Resistor_SMD:R_0603"
+		(property "Footprint" "V2_Resistor_SMD:R_1608"
 			(at 86.36 183.388 0)
 			(hide yes)
@@
 	)
 	(symbol
-		(lib_id "V2_Capacitor:0603_10u")
+		(lib_id "V2_Capacitor:1608_10u")
 		(at 64.77 151.13 0)
 		(unit 1)
@@
 			)
 		)
-		(property "Footprint" "V2_Capacitor_SMD:C_0603"
+		(property "Footprint" "V2_Capacitor_SMD:C_1608"
 			(at 64.77 168.148 0)
 			(hide yes)
@@
 	)
 	(symbol
-		(lib_id "V2_Capacitor:0603_1u")
+		(lib_id "V2_Capacitor:1608_1u")
 		(at 95.25 24.13 0)
 		(unit 1)
@@
 			)
 		)
-		(property "Footprint" "V2_Capacitor_SMD:C_0603"
+		(property "Footprint" "V2_Capacitor_SMD:C_1608"
 			(at 95.25 41.148 0)
 			(hide yes)
@@
 	)
 	(symbol
-		(lib_id "V2_Resistor:0603_100k")
+		(lib_id "V2_Resistor:1608_100k")
 		(at 57.15 123.19 90)
 		(unit 1)
@@
 			)
 		)
-		(property "Footprint" "V2_Resistor_SMD:R_0603"
+		(property "Footprint" "V2_Resistor_SMD:R_1608"
 			(at 72.898 123.19 0)
 			(hide yes)

Commit message: Refresh
Parts:
- D101: footprint V2_LED:LED_0603 -> V2_LED:LED_1608
Changed lines of the file:
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@@
 	(title_block
 		(title "V2 axis")
-		(date "2026-04-23")
+		(date "2026-05-19")
 		(rev "2026-01-14")
 		(company "Versio Duo")
@@
 			)
 		)
-		(property "Footprint" "V2_LED:LED_0603"
+		(property "Footprint" "V2_LED:LED_1608"
 			(at 127 54.61 90)
 			(hide yes)
@@
 		(unit 1)
 		(body_style 1)
-		(exclude_from_sim no)
+		(exclude_from_sim yes)
 		(in_bom no)
 		(on_board yes)
@@
 			)
 		)
-		(property "Sim.Enable" "0"
-			(at 234.95 152.4 0)
-			(hide yes)
-			(show_name no)
-			(do_not_autoplace no)
-			(effects
-				(font
-					(size 1.27 1.27)
-				)
-			)
-		)
 		(instances
 			(project "axis"
@@
 		(unit 1)
 		(body_style 1)
-		(exclude_from_sim no)
+		(exclude_from_sim yes)
 		(in_bom no)
 		(on_board yes)
@@
 			(at 176.53 165.1 0)
 			(hide yes)
-			(show_name no)
-			(do_not_autoplace no)
-			(effects
-				(font
-					(size 1.27 1.27)
-				)
-			)
-		)
-		(property "Sim.Enable" "0"
-			(at 176.53 165.1 0)
-			(hide yes)

Commit message: Refresh
Parts:
- INFO102: value Layer_Numbers -> Layer_Numbers-4; footprint V2_Production:Layer_Numbers -> V2_Production:Layer_Numbers-4; symbol V2_Production:Layer_Numbers -> V2_Production:Layer_Numbers-4
Changed lines of the file:
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@@
 	(title_block
 		(title "V2 axis")
-		(date "2026-05-19")
+		(date "2026-05-27")
 		(rev "2026-01-14")
 		(company "Versio Duo")
@@
 				(font
 					(size 1.27 1.27)
+					(color 255 92 187 1)
 				)
 			)
@@
 		(in_pos_files yes)
 		(dnp no)
-		(fields_autoplaced yes)
 		(property "Reference" "#PWR0136"
 			(at 242.57 76.2 0)
@@
 		)
 		(property "Value" "+5V"
-			(at 250.19 76.1999 90)
+			(at 252.984 76.1999 90)
 			(show_name no)
 			(do_not_autoplace no)
@@
 				(font
 					(size 1.27 1.27)
+					(color 255 92 187 1)
 				)
-				(justify left)
 			)
 		)
@@
 		)
 		(property "Value" "+5V"
-			(at 265.43 101.5999 90)
+			(at 267.97 101.5999 90)
 			(show_name no)
 			(do_not_autoplace no)
@@
 				(font
 					(size 1.27 1.27)
+					(color 255 92 187 1)
 				)
-				(justify left)
 			)
 		)
@@
 				(font
 					(size 1.27 1.27)
+					(color 255 92 187 1)
 				)
 			)
@@
 		)
 		(property "Value" "+5V"
-			(at 276.86 40.6399 0)
+			(at 275.59 40.8939 0)
 			(show_name no)
 			(do_not_autoplace no)
@@
 				(font
 					(size 1.27 1.27)
+					(color 255 92 187 1)
 				)
-				(justify right)
 			)
 		)
@@
 		(in_pos_files yes)
 		(dnp no)
-		(fields_autoplaced yes)
 		(property "Reference" "#PWR0105"
 			(at 58.42 123.19 0)
@@
 		)
 		(property "Value" "+3V3"
-			(at 50.8 123.1899 90)
+			(at 48.26 123.1899 90)
 			(show_name no)
 			(do_not_autoplace no)
@@
 				(font
 					(size 1.27 1.27)
+					(color 255 92 187 1)
 				)
-				(justify left)
 			)
 		)
@@
 		(in_pos_files yes)
 		(dnp no)
-		(fields_autoplaced yes)
 		(property "Reference" "#PWR0106"
 			(at 63.5 48.26 0)
@@
 		)
 		(property "Value" "+3V3"
-			(at 55.88 48.2599 90)
+			(at 53.34 48.2599 90)
 			(show_name no)
 			(do_not_autoplace no)
@@
 				(font
 					(size 1.27 1.27)
+					(color 255 92 187 1)
 				)
-				(justify left)
 			)
 		)
@@
 		)
 		(property "Value" "+3V3"
-			(at 59.69 144.78 0)
+			(at 59.69 143.764 0)
 			(show_name no)
 			(do_not_autoplace no)
@@
 				(font
 					(size 1.27 1.27)
+					(color 255 92 187 1)
 				)
 			)
@@
 				(font
 					(size 1.27 1.27)
+					(color 255 92 187 1)
 				)
 			)
@@
 		(in_pos_files yes)
 		(dnp no)
-		(fields_autoplaced yes)
 		(property "Reference" "#PWR0116"
 			(at 118.11 96.52 0)
@@
 		)
 		(property "Value" "+3V3"
-			(at 110.49 96.5199 90)
+			(at 107.696 96.5199 90)
 			(show_name no)
 			(do_not_autoplace no)
@@
 				(font
 					(size 1.27 1.27)
+					(color 255 92 187 1)
 				)
-				(justify left)
 			)
 		)
@@
 	)
 	(symbol
-		(lib_id "V2_Production:Layer_Numbers")
+		(lib_id "V2_Production:Layer_Numbers-4")
 		(at 176.53 180.34 0)
 		(unit 1)
@@
 			)
 		)
-		(property "Value" "Layer_Numbers"
+		(property "Value" "Layer_Numbers-4"
 			(at 178.4684 176.8685 0)
 			(hide yes)
@@
 			)
 		)
-		(property "Footprint" "V2_Production:Layer_Numbers"
+		(property "Footprint" "V2_Production:Layer_Numbers-4"
 			(at 176.53 186.69 0)
 			(hide yes)
@@
 		)
 		(property "Value" "Shield"
-			(at 253.238 83.82 90)
+			(at 255.778 83.82 90)
 			(show_name no)
 			(do_not_autoplace no)
@@
 		(in_pos_files yes)
 		(dnp no)
-		(fields_autoplaced yes)
 		(property "Reference" "#PWR0131"
 			(at 195.58 90.17 0)
@@
 		)
 		(property "Value" "+5V"
-			(at 203.2 90.1699 90)
+			(at 205.232 90.1699 90)
 			(show_name no)
 			(do_not_autoplace no)
@@
 				(font
 					(size 1.27 1.27)
+					(color 255 92 187 1)
 				)
-				(justify left)
 			)
 		)
@@
 				(font
 					(size 1.27 1.27)
+					(color 255 92 187 1)
 				)
 			)
@@
 		)
 		(property "Value" "+3V3"
-			(at 85.09 161.29 0)
+			(at 85.09 160.528 0)
 			(show_name no)
 			(do_not_autoplace no)
@@
 				(font
 					(size 1.27 1.27)
+					(color 255 92 187 1)
 				)
 			)
@@
 		)
 		(property "Value" "+3V3"
-			(at 31.75 151.13 0)
+			(at 31.75 150.368 0)
 			(show_name no)
 			(do_not_autoplace no)
@@
 				(font
 					(size 1.27 1.27)
+					(color 255 92 187 1)
 				)
 			)
@@
 		)
 		(property "Value" "+3V3"
-			(at 119.38 177.165 90)
+			(at 119.126 177.673 90)
 			(show_name no)
 			(do_not_autoplace no)
@@
 				(font
 					(size 1.27 1.27)
+					(color 255 92 187 1)
 				)
 			)
