File: hardware/front/front.kicad_pcb (KiCad board)
At the start: 2 copper layers, 66 x 17.5 mm, 0 parts

Commit message: Rounded edge
Other:
- board size 66 x 17.5 mm -> 70 x 17.5 mm
Changed lines of the file:
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@@
 (kicad_pcb
-	(version 20241229)
+	(version 20260206)
 	(generator "pcbnew")
-	(generator_version "9.0")
+	(generator_version "10.0")
 	(general
-		(thickness 2.09)
+		(thickness 2)
 		(legacy_teardrops no)
 	)
@@
 			(layer "F.Mask"
 				(type "Top Solder Mask")
-				(thickness 0.01)
+				(thickness 0)
 			)
 			(layer "F.Cu"
 				(type "copper")
-				(thickness 0.035)
+				(thickness 0)
 			)
 			(layer "dielectric 1"
@@
 			(layer "B.Cu"
 				(type "copper")
-				(thickness 0.035)
+				(thickness 0)
 			)
 			(layer "B.Mask"
 				(type "Bottom Solder Mask")
-				(thickness 0.01)
+				(thickness 0)
 			)
 			(layer "B.Paste"
@@
 		(pad_to_mask_clearance 0)
 		(allow_soldermask_bridges_in_footprints no)
-		(tenting front back)
+		(tenting
+			(front yes)
+			(back yes)
+		)
+		(covering
+			(front no)
+			(back no)
+		)
+		(plugging
+			(front no)
+			(back no)
+		)
+		(capping no)
+		(filling no)
 		(aux_axis_origin 60 125)
 		(grid_origin 60 125)
@@
 			(usegerberadvancedattributes yes)
 			(creategerberjobfile yes)
-			(dashed_line_dash_ratio 12.000000)
-			(dashed_line_gap_ratio 3.000000)
+			(dashed_line_dash_ratio 12)
+			(dashed_line_gap_ratio 3)
 			(svgprecision 4)
 			(plotframeref no)
 			(mode 1)
 			(useauxorigin no)
-			(hpglpennumber 1)
-			(hpglpenspeed 20)
-			(hpglpendiameter 15.000000)
 			(pdf_front_fp_property_popups yes)
 			(pdf_back_fp_property_popups yes)
@@
 		)
 	)
-	(net 0 "")
+	(gr_line
+		(start 60 108.5)
+		(end 60 124)
+		(stroke
+			(width 0.05)
+			(type solid)
+		)
+		(layer "Edge.Cuts")
+	)
 	(gr_arc
 		(start 60 108.5)
@@
 	)
 	(gr_line
-		(start 60 108.5)
-		(end 60 124)
-		(stroke
-			(width 0.05)
-			(type solid)
-		)
-		(layer "Edge.Cuts")
-	)
-	(gr_line
-		(start 61 125)
-		(end 125 125)
-		(stroke
-			(width 0.05)
-			(type solid)
-		)
-		(layer "Edge.Cuts")
-	)
-	(gr_circle
-		(center 112 116.25)
-		(end 113.1 116.25)
-		(stroke
-			(width 0.05)
-			(type solid)
-		)
-		(fill no)
-		(layer "Edge.Cuts")
-	)
-	(gr_arc
-		(start 125 107.5)
-		(mid 125.707107 107.792893)
-		(end 126 108.5)
-		(stroke
-			(width 0.05)
-			(type solid)
-		)
-		(layer "Edge.Cuts")
-	)
-	(gr_arc
-		(start 126 124)
-		(mid 125.707107 124.707107)
-		(end 125 125)
-		(stroke
-			(width 0.05)
-			(type solid)
-		)
-		(layer "Edge.Cuts")
-	)
-	(gr_line
 		(start 61 107.5)
-		(end 125 107.5)
-		(stroke
-			(width 0.05)
-			(type solid)
-		)
-		(layer "Edge.Cuts")
-	)
-	(gr_line
-		(start 126 108.5)
-		(end 126 124)
-		(stroke
-			(width 0.05)
-			(type solid)
-		)
-		(layer "Edge.Cuts")
-	)
-	(gr_circle
-		(center 97.5 111.25)
-		(end 98 111.25)
-		(stroke
-			(width 0.05)
-			(type solid)
-		)
-		(fill no)
+		(end 121.25 107.5)
+		(stroke
+			(width 0.05)
+			(type solid)
+		)
 		(layer "Edge.Cuts")
 	)
@@
 		(layer "Edge.Cuts")
 	)
+	(gr_line
+		(start 61 125)
+		(end 121.25 125)
+		(stroke
+			(width 0.05)
+			(type solid)
+		)
+		(layer "Edge.Cuts")
+	)
 	(gr_circle
 		(center 74 116.25)
@@
 		(layer "Edge.Cuts")
 	)
+	(gr_circle
+		(center 97.5 111.25)
+		(end 98 111.25)
+		(stroke
+			(width 0.05)
+			(type solid)
+		)
+		(fill no)
+		(layer "Edge.Cuts")
+	)
+	(gr_circle
+		(center 112 116.25)
+		(end 113.1 116.25)
+		(stroke
+			(width 0.05)
+			(type solid)
+		)
+		(fill no)
+		(layer "Edge.Cuts")
+	)
+	(gr_arc
+		(start 121.25 107.5)
+		(mid 130 116.25)
+		(end 121.25 125)
+		(stroke
+			(width 0.05)
+			(type solid)
+		)
+		(layer "Edge.Cuts")
+	)
